File: pcb/usb-ri.brd (EAGLE design)
At the start: 44 x 44 mm, 43 parts, among them IC1 STM32F303, IC2 REG1117, IC3 STF203-22, IC4 FT231XS-R, J1 JTAG, J2 MJ-3536, J3 RESET, J4 10118193-0001LF, Q1 IRLML9303, Q2 IRLML2030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

Commit message: Fixed PCB bug: connection of USB port
Connections:
- net GND: now also J4.5; no longer J4.4
